File: hw/KELU1-0232.brd (EAGLE design)
At the start: 117 x 121 mm, 219 parts, among them IC1 FSBB30CH60, IC10 LM358D, IC11 LM358D, IC12 IL3000, IC13 HCPL-3180-300E, IC14 HCPL-3180-300E, IC15 74AC14D, IC17 L78MXXAB, IC19 MC34063AD, IC2 4049D, IC3 LM358D, IC4 LM358D, IC5 LM358D, IC6 LM358D, IC7 IL3000, IC8 IL3000, IC9 IL3000, K3 HJR-21FF, P1 B3B-EH-A, P2 B3B-EH-A, P3 B3B-EH-A, P4 B3B-EH-A, P5 B3B-EH-A, P6 B3B-EH-A, Q1 BC817-16LT1SMD, Q2 IRFP240-H, Q3 BC817-40SMD, X1 DG129-7.5-02P, X2 DG129-7.5-02P, X3 DG129-7.5-03P, X4 DG129-7.5-02P

Commit message: refresh
refresh
Parts:
- added J1: 0480251190, Connectors:JACK
Routing:
- net +5VA: track 250.8 -> 250.9 mm, vias 11 -> 10
Changed lines of the file:
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@@
 <?xml version="1.0" encoding="utf-8"?>
 <!DOCTYPE eagle SYSTEM "eagle.dtd">
-<eagle version="7.6.0">
+<eagle version="9.0.0">
 <drawing>
 <settings>
 <setting alwaysvectorfont="no"/>
+<setting keepoldvectorfont="yes"/>
 <setting verticaltext="up"/>
 </settings>
@@
 <layer number="52" name="bDocu" color="7" fill="1" visible="yes" active="yes"/>
 <layer number="56" name="wert" color="7" fill="1" visible="no" active="yes"/>
+<layer number="57" name="t3Ddata" color="7" fill="1" visible="yes" active="yes"/>
+<layer number="58" name="b3Ddata" color="7" fill="1" visible="yes" active="yes"/>
+<layer number="88" name="SimResults" color="9" fill="1" visible="no" active="no"/>
+<layer number="89" name="SimProbes" color="9" fill="1" visible="no" active="no"/>
 <layer number="90" name="Modules" color="5" fill="1" visible="no" active="no"/>
 <layer number="91" name="Nets" color="2" fill="1" visible="no" active="no"/>
@@
 <param name="dpMaxLengthDifference" value="10mm"/>
 <param name="dpGapFactor" value="2.5"/>
-<param name="checkGrid" value="0"/>
 <param name="checkAngle" value="0"/>
 <param name="checkFont" value="1"/>
 <param name="checkRestrict" value="1"/>
+<param name="checkStop" value="0"/>
+<param name="checkValues" value="0"/>
 <param name="useDiameter" value="13"/>
 <param name="maxErrors" value="50"/>
@@
 <element name="C44" library="resistor" package="C1206" value="" x="73" y="89"/>
 <element name="IC13" library="HCPL-3180-300E" package="HCPL-3180" value="HCPL-3180-300E" x="35.5" y="37">
-<attribute name="MOUSER_PRICE-STOCK" value="https://www.mouser.com/Search/Refine.aspx?Keyword=630-HCPL-3180-300E" x="35.5" y="37" size="1.778" layer="27" display="off"/>
+<attribute name="DESCRIPTION" value="Broadcom HCPL-3180-300E DC Input IGBT Gate Drive Output Dual Optocoupler, Surface Mount, 8-Pin DIP" x="35.5" y="37" size="1.778" layer="27" display="off"/>
+<attribute name="HEIGHT" value="mm" x="35.5" y="37" size="1.778" layer="27" display="off"/>
 <attribute name="MANUFACTURER_NAME" value="Avago Technologies" x="35.5" y="37" size="1.778" layer="27" display="off"/>
 <attribute name="MANUFACTURER_PART_NUMBER" value="HCPL-3180-300E" x="35.5" y="37" size="1.778" layer="27" display="off"/>
 <attribute name="MOUSER_PART_NUMBER" value="630-HCPL-3180-300E" x="35.5" y="37" size="1.778" layer="27" display="off"/>
+<attribute name="MOUSER_PRICE-STOCK" value="https://www.mouser.com/Search/Refine.aspx?Keyword=630-HCPL-3180-300E" x="35.5" y="37" size="1.778" layer="27" display="off"/>
 <attribute name="RS_PART_NUMBER" value="8188347P" x="35.5" y="37" size="1.778" layer="27" display="off"/>
-<attribute name="DESCRIPTION" value="Broadcom HCPL-3180-300E DC Input IGBT Gate Drive Output Dual Optocoupler, Surface Mount, 8-Pin DIP" x="35.5" y="37" size="1.778" layer="27" display="off"/>
-<attribute name="HEIGHT" value="mm" x="35.5" y="37" size="1.778" layer="27" display="off"/>
 <attribute name="RS_PRICE-STOCK" value="http://uk.rs-online.com/web/p/products/8188347P" x="35.5" y="37" size="1.778" layer="27" display="off"/>
 </element>
 <element name="IC14" library="HCPL-3180-300E" package="HCPL-3180" value="HCPL-3180-300E" x="24.5" y="37">
-<attribute name="MOUSER_PRICE-STOCK" value="https://www.mouser.com/Search/Refine.aspx?Keyword=630-HCPL-3180-300E" x="24.5" y="37" size="1.778" layer="27" display="off"/>
+<attribute name="DESCRIPTION" value="Broadcom HCPL-3180-300E DC Input IGBT Gate Drive Output Dual Optocoupler, Surface Mount, 8-Pin DIP" x="24.5" y="37" size="1.778" layer="27" display="off"/>
+<attribute name="HEIGHT" value="mm" x="24.5" y="37" size="1.778" layer="27" display="off"/>
 <attribute name="MANUFACTURER_NAME" value="Avago Technologies" x="24.5" y="37" size="1.778" layer="27" display="off"/>
 <attribute name="MANUFACTURER_PART_NUMBER" value="HCPL-3180-300E" x="24.5" y="37" size="1.778" layer="27" display="off"/>
 <attribute name="MOUSER_PART_NUMBER" value="630-HCPL-3180-300E" x="24.5" y="37" size="1.778" layer="27" display="off"/>
+<attribute name="MOUSER_PRICE-STOCK" value="https://www.mouser.com/Search/Refine.aspx?Keyword=630-HCPL-3180-300E" x="24.5" y="37" size="1.778" layer="27" display="off"/>
 <attribute name="RS_PART_NUMBER" value="8188347P" x="24.5" y="37" size="1.778" layer="27" display="off"/>
-<attribute name="DESCRIPTION" value="Broadcom HCPL-3180-300E DC Input IGBT Gate Drive Output Dual Optocoupler, Surface Mount, 8-Pin DIP" x="24.5" y="37" size="1.778" layer="27" display="off"/>
-<attribute name="HEIGHT" value="mm" x="24.5" y="37" size="1.778" layer="27" display="off"/>
 <attribute name="RS_PRICE-STOCK" value="http://uk.rs-online.com/web/p/products/8188347P" x="24.5" y="37" size="1.778" layer="27" display="off"/>
 </element>
@@
 </element>
 <element name="K3" library="HJR-21FF" package="HJR21FF" value="HJR-21FF" x="16.25" y="99.25" rot="MR0"/>
+<element name="J1" library="Connectors" library_urn="urn:adsk.eagle:library:14555660" package="JACK" package3d_urn="urn:adsk.eagle:package:10989918/4" value="0480251190" x="4" y="-36">
+<attribute name="CREATED_BY" value="PCBLayout.com" x="4" y="-36" size="1.778" layer="27" display="off"/>
+<attribute name="DIGIKEY_PART_NUMBER" value="WM5484-ND" x="4" y="-36" size="1.778" layer="27" display="off"/>
+<attribute name="MANUFACTURER" value="Molex" x="4" y="-36" size="1.778" layer="27" display="off"/>
+<attribute name="MPN" value="0480251190" x="4" y="-36" size="1.778" layer="27" display="off"/>
+</element>
 </elements>
 <signals>
@@
 <wire x1="78" y1="14.75" x2="81.365" y2="18.115" width="0.3048" layer="1"/>
 <wire x1="81.365" y1="18.115" x2="81.365" y2="19.35" width="0.3048" layer="1"/>
-<wire x1="66.95" y1="14.75" x2="66.93" y2="14.73" width="0" layer="19" extent="1-1"/>
+<wire x1="66.93" y1="14.73" x2="66.95" y2="14.75" width="0.1524" layer="1"/>
 </signal>
 <signal name="N$63">
@@
 <wire x1="99" y1="9.75" x2="99" y2="20.75" width="0.6096" layer="16"/>
 <wire x1="99" y1="20.75" x2="99.27" y2="20.77" width="0.6096" layer="16"/>
-<wire x1="100.56" y1="20.75" x2="99" y2="20.75" width="0.6096" layer="16"/>
+<wire x1="100.06" y1="20.75" x2="99" y2="20.75" width="0.6096" layer="16"/>
 <wire x1="99" y1="20.75" x2="99" y2="31.75" width="0.6096" layer="16"/>
 <wire x1="99" y1="31.75" x2="99.27" y2="31.77" width="0.6096" layer="16"/>
@@
 <wire x1="53.75" y1="39.5" x2="63.25" y2="39.5" width="0.6096" layer="16"/>
 <wire x1="63.25" y1="39.5" x2="64.75" y2="39.5" width="0.6096" layer="16"/>
-<wire x1="42.69" y1="40.81" x2="42.75" y2="40.81" width="0.6096" layer="16"/>
 <wire x1="42.75" y1="40.81" x2="42.75" y2="39.5" width="0.6096" layer="16"/>
 <wire x1="42.75" y1="39.5" x2="51.75" y2="39.5" width="0.6096" layer="16"/>
@@
 <wire x1="51.25" y1="43.5" x2="51.75" y2="43" width="0.3048" layer="16"/>
 <wire x1="51.75" y1="43" x2="51.75" y2="39.5" width="0.3048" layer="16"/>
-<via x="42.75" y="40.87" extent="1-16" drill="0.3"/>
-<wire x1="42.75" y1="40.87" x2="42.75" y2="44.4" width="0.3048" layer="1"/>
+<wire x1="42.75" y1="41.37" x2="42.75" y2="44.4" width="0.3048" layer="1"/>
 <wire x1="42.75" y1="44.4" x2="42.85" y2="44.5" width="0.3048" layer="1"/>
 <wire x1="42.85" y1="44.5" x2="42.85" y2="45.15" width="0.3048" layer="1"/>
@@
 <wire x1="100.58" y1="20.77" x2="105.02" y2="20.77" width="0.4064" layer="16"/>
 <wire x1="105.02" y1="20.77" x2="105.5" y2="21.25" width="0.4064" layer="16"/>
-<wire x1="100.56" y1="20.75" x2="100.58" y2="20.77" width="0" layer="19" extent="16-16"/>
+<wire x1="100.58" y1="20.77" x2="100.08" y2="20.77" width="0.1524" layer="16"/>
+<wire x1="100.08" y1="20.77" x2="100.06" y2="20.75" width="0.1524" layer="16"/>
+<wire x1="42.69" y1="40.81" x2="42.75" y2="40.81" width="0.1524" layer="16"/>
+<wire x1="42.69" y1="40.81" x2="42.69" y2="41.31" width="0.1524" layer="1"/>
+<wire x1="42.69" y1="41.31" x2="42.75" y2="41.37" width="0.1524" layer="1"/>
 </signal>
 <signal name="+5V">
@@
 </board>
 </drawing>
+<compatibility>
+<note version="8.2" severity="warning">
+Since Version 8.2, EAGLE supports online libraries. The ids
+of those online libraries will not be understood (or retained)
+with this version.
+</note>
+<note version="8.3" severity="warning">
+Since Version 8.3, EAGLE supports URNs for individual library
+assets (packages, symbols, and devices). The URNs of those assets
+will not be understood (or retained) with this version.
+</note>
+<note version="8.3" severity="warning">
+Since Version 8.3, EAGLE supports the association of 3D packages
+with devices in libraries, schematics, and board files. Those 3D
+packages will not be understood (or retained) with this version.
+</note>
+</compatibility>
 </eagle>
