File: hw/KELU1-0232.sch (EAGLE design)
At the start: 213 parts, among them IC1 FSBB30CH60, IC10 LM358D, IC11 LM358D, IC12 IL3000, IC13 HCPL-3180-300E, IC14 HCPL-3180-300E, IC15 74AC14D, IC17 L78MXXAB, IC19 MC34063AD, IC2 4049D, IC3 LM358D, IC4 LM358D, IC5 LM358D, IC6 LM358D, IC7 IL3000, IC8 IL3000, IC9 IL3000, K3 HJR-21FF, P1 B3B-EH-A, P2 B3B-EH-A, P3 B3B-EH-A, P4 B3B-EH-A, P5 B3B-EH-A, P6 B3B-EH-A, Q1 BC817-16LT1SMD, Q2 IRFP240-H, Q3 BC817-40SMD, X1 DG129-7.5-02P, X2 DG129-7.5-02P, X3 DG129-7.5-03P, X4 DG129-7.5-02P

Commit message: refresh
refresh
Parts:
- added J1: 0480251190, Connectors:0480251190
Changed lines of the file:
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@@
 <?xml version="1.0" encoding="utf-8"?>
 <!DOCTYPE eagle SYSTEM "eagle.dtd">
-<eagle version="7.6.0">
+<eagle version="9.0.0">
 <drawing>
 <settings>
 <setting alwaysvectorfont="no"/>
+<setting keepoldvectorfont="yes"/>
 <setting verticaltext="up"/>
 </settings>
-<grid distance="0.1" unitdist="inch" unit="inch" style="lines" multiple="1" display="yes" altdistance="0.01" altunitdist="inch" altunit="inch"/>
+<grid distance="0.1" unitdist="inch" unit="inch" style="lines" multiple="1" display="no" altdistance="0.01" altunitdist="inch" altunit="inch"/>
 <layers>
 <layer number="1" name="Top" color="4" fill="1" visible="no" active="no"/>
@@
 <layer number="52" name="bDocu" color="7" fill="1" visible="no" active="no"/>
 <layer number="56" name="wert" color="7" fill="1" visible="no" active="no"/>
+<layer number="88" name="SimResults" color="9" fill="1" visible="yes" active="yes"/>
+<layer number="89" name="SimProbes" color="9" fill="1" visible="yes" active="yes"/>
 <layer number="90" name="Modules" color="5" fill="1" visible="no" active="yes"/>
 <layer number="91" name="Nets" color="2" fill="1" visible="yes" active="yes"/>
@@
 <part name="X4" library="DG129" deviceset="DG129-7.5-02P" device=""/>
 <part name="K3" library="HJR-21FF" deviceset="HJR-21FF" device=""/>
+<part name="J1" library="Connectors" library_urn="urn:adsk.eagle:library:14555660" deviceset="0480251190" device="" package3d_urn="urn:adsk.eagle:package:10989918/4"/>
 </parts>
 <sheets>
@@
 <instance part="X3" gate="-2" x="210.82" y="157.48" rot="R90"/>
 <instance part="X3" gate="-3" x="218.44" y="157.48" rot="R90"/>
+<instance part="J1" gate="G$1" x="190.5" y="63.5"/>
 </instances>
 <busses>
@@
 </schematic>
 </drawing>
+<compatibility>
+<note version="8.2" severity="warning">
+Since Version 8.2, EAGLE supports online libraries. The ids
+of those online libraries will not be understood (or retained)
+with this version.
+</note>
+<note version="8.3" severity="warning">
+Since Version 8.3, EAGLE supports URNs for individual library
+assets (packages, symbols, and devices). The URNs of those assets
+will not be understood (or retained) with this version.
+</note>
+<note version="8.3" severity="warning">
+Since Version 8.3, EAGLE supports the association of 3D packages
+with devices in libraries, schematics, and board files. Those 3D
+packages will not be understood (or retained) with this version.
+</note>
+</compatibility>
 </eagle>
